File: SiPMT revA/SiPMT.revA.kicad_pcb (KiCad board)
At the start: 2 copper layers, 55.6 x 69 mm, 150 parts

Commit message: Updated the layers and resistors
Parts:
- moved R8 1.69 mm to (171.2, 68.2), turned to 0 degrees
- moved R31 1.69 mm to (171.2, 82.2), turned to 0 degrees
- moved R32 1.69 mm to (171.2, 89.2), turned to 0 degrees
- moved R47 1.69 mm to (171.2, 96.2), turned to 0 degrees
- moved R48 1.69 mm to (171.2, 103.2), turned to 0 degrees
- moved R63 1.69 mm to (171.2, 110.2), turned to 0 degrees
- moved R64 1.69 mm to (171.2, 117.2), turned to 0 degrees
- moved R9 1.69 mm to (171.2, 75.2), turned to 0 degrees
- moved Q2 0.80 mm to (141.3, 126.7)
- moved Q3 0.80 mm to (132.6, 126.7)
- moved C4 0.80 mm to (130.3, 123.6)
- moved C5 0.80 mm to (139.1, 123.6)
- moved C6 0.80 mm to (163.4, 123.6)
- moved C7 0.80 mm to (154.7, 123.6)
- moved H10 0.80 mm to (165.3, 126.6)
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- renumbered H11 to Q1, H12 to Q2, H14 to Q3, H13 to Q4
Routing:
- net +BATT 4: track 6.60 -> 31.7 mm, vias 1 -> 14
- net +BATT 3: track 6.07 -> 30.9 mm, vias 1 -> 18
- net +BATT 1: track 44.6 -> 67.3 mm, vias 1 -> 14
- net +BATT 2: track 41.5 -> 62.8 mm, vias 1 -> 18
- net GND: track 14.0 -> 0.00 mm, vias 0 -> 34
- net /AE3_CH5: track 17.1 -> 12.6 mm
- net /AE3_CH0: track 15.2 -> 14.5 mm
- added copper zone on In2.Cu, net +BATT 1
- added copper zone on In2.Cu, net +BATT 2
- added copper zone on In2.Cu, net +BATT 3
- added copper zone on In2.Cu, net +BATT 4
- added copper zone on B.Cu, net GND
- added copper zone on In1.Cu, net GND
- removed copper zone on B.Cu, net +BATT 1
- removed copper zone on B.Cu, net +BATT 2
- removed copper zone on B.Cu, net +BATT 3
- removed copper zone on B.Cu, net +BATT 4
Other:
- copper layers 2 -> 4
- board text added: "Jacob Romeo Varner Lab 2024-10-28"
- board text added: "Q1"
- board text added: "Q2"
- board text added: "Q3"
- board text added: "Q4"
- board text added: "add vias to VCC res"
- board text removed: "2024-09-30"
- board text removed: "IDL_24_032"

Commit message: updated gerber files
Other:
- board text removed: "add vias to VCC res"
Changed lines of the file:
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@@
 		(layer "User.6")
-	)
-	(gr_text "\nadd vias to VCC res"
-		(at 183.9 93.93 0)
-		(layer "F.Cu")
-		(effects
-			(font
-				(size 1.5 1.5)
-				(thickness 0.3)
-				(bold yes)
-			)
-			(justify left bottom)
-		)
 	)
 	(gr_text "Q3"

Commit message: updated name
Routing:
- net +BATT 4: vias 14 -> 13
- net +BATT 3: vias 18 -> 17
- net +BATT 2: vias 18 -> 17
- net +BATT 1: vias 14 -> 13
Other:
- board text added: "IDL_24_032"
- board text added: "Jacob Romeo Varner Lab 2024-11-25"
- board text removed: "Jacob Romeo Varner Lab 2024-10-28"
Changed lines of the file:
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@@
 		(tags "mounting hole 2.5mm")
 		(property "Reference" "Q3"
-			(at 0 2.3 -0)
+			(at 0 2.3 0)
 			(layer "B.SilkS")
 			(effects
@@
 		(tags "mounting hole 2.5mm")
 		(property "Reference" "Q4"
-			(at 0 2.325 -0)
+			(at 0 2.325 0)
 			(layer "B.SilkS")
 			(effects
@@
 		)
 		(pad "1" thru_hole circle
-			(at 0.05 0)
+			(at 0 0)
 			(size 5 5)
 			(drill 2.5)
@@
 		(tags "mounting hole 2.5mm")
 		(property "Reference" "Q2"
-			(at 0 2.35 -0)
+			(at 0 2.35 0)
 			(layer "B.SilkS")
 			(effects
@@
 		(tags "mounting hole 2.5mm")
 		(property "Reference" "Q1"
-			(at 0.05 2.325 -0)
+			(at 0.05 2.325 0)
 			(layer "B.SilkS")
 			(effects
@@
 		(tags "resistor handsolder")
 		(property "Reference" "R48"
-			(at 1.45 0 360)
+			(at 1.45 0 0)
 			(layer "B.SilkS")
 			(hide yes)
@@
 		)
 		(property "Value" "10k"
-			(at 0 -1.43 360)
+			(at 0 -1.43 0)
 			(layer "B.Fab")
 			(hide yes)
@@
 		)
 		(property "Footprint" "kicad-mza:0603"
-			(at 0.175 -1.5 360)
+			(at 0.175 -1.5 0)
 			(layer "B.Fab")
 			(hide yes)
@@
 		)
 		(property "Datasheet" ""
-			(at 0 0 360)
+			(at 0 0 0)
 			(layer "B.Fab")
 			(hide yes)
@@
 		)
 		(property "Description" "Resistor"
-			(at 0 0 360)
+			(at 0 0 0)
 			(layer "B.Fab")
 			(hide yes)
@@
 		(tags "resistor handsolder")
 		(property "Reference" "R8"
-			(at 1.45 0 360)
+			(at 1.45 0 0)
 			(layer "B.SilkS")
 			(hide yes)
@@
 		)
 		(property "Value" "10k"
-			(at 0 -1.43 360)
+			(at 0 -1.43 0)
 			(layer "B.Fab")
 			(hide yes)
@@
 		)
 		(property "Footprint" "kicad-mza:0603"
-			(at 0.175 -1.5 360)
+			(at 0.175 -1.5 0)
 			(layer "B.Fab")
 			(hide yes)
@@
 		)
 		(property "Datasheet" ""
-			(at 0 0 360)
+			(at 0 0 0)
 			(layer "B.Fab")
 			(hide yes)
@@
 		)
 		(property "Description" "Resistor"
-			(at 0 0 360)
+			(at 0 0 0)
 			(layer "B.Fab")
 			(hide yes)
@@
 		(tags "resistor handsolder")
 		(property "Reference" "R47"
-			(at 1.45 0 360)
+			(at 1.45 0 0)
 			(layer "B.SilkS")
 			(hide yes)
@@
 		)
 		(property "Value" "10k"
-			(at 0 -1.43 360)
+			(at 0 -1.43 0)
 			(layer "B.Fab")
 			(hide yes)
@@
 		)
 		(property "Footprint" "kicad-mza:0603"
-			(at 0.175 -1.5 360)
+			(at 0.175 -1.5 0)
 			(layer "B.Fab")
 			(hide yes)
@@
 		)
 		(property "Datasheet" ""
-			(at 0 0 360)
+			(at 0 0 0)
 			(layer "B.Fab")
 			(hide yes)
@@
 		)
 		(property "Description" "Resistor"
-			(at 0 0 360)
+			(at 0 0 0)
 			(layer "B.Fab")
 			(hide yes)
@@
 		(tags "resistor handsolder")
 		(property "Reference" "R63"
-			(at 1.45 0 360)
+			(at 1.45 0 0)
 			(layer "B.SilkS")
 			(hide yes)
@@
 		)
 		(property "Value" "10k"
-			(at 0 -1.43 360)
+			(at 0 -1.43 0)
 			(layer "B.Fab")
 			(hide yes)
@@
 		)
 		(property "Footprint" "kicad-mza:0603"
-			(at 0.175 -1.5 360)
+			(at 0.175 -1.5 0)
 			(layer "B.Fab")
 			(hide yes)
@@
 		)
 		(property "Datasheet" ""
-			(at 0 0 360)
+			(at 0 0 0)
 			(layer "B.Fab")
 			(hide yes)
@@
 		)
 		(property "Description" "Resistor"
-			(at 0 0 360)
+			(at 0 0 0)
 			(layer "B.Fab")
 			(hide yes)
@@
 		(tags "resistor handsolder")
 		(property "Reference" "R9"
-			(at 1.45 0 360)
+			(at 1.45 0 0)
 			(layer "B.SilkS")
 			(hide yes)
@@
 		)
 		(property "Value" "10k"
-			(at 0 -1.43 360)
+			(at 0 -1.43 0)
 			(layer "B.Fab")
 			(hide yes)
@@
 		)
 		(property "Footprint" "kicad-mza:0603"
-			(at 0.175 -1.5 360)
+			(at 0.175 -1.5 0)
 			(layer "B.Fab")
 			(hide yes)
@@
 		)
 		(property "Datasheet" ""
-			(at 0 0 360)
+			(at 0 0 0)
 			(layer "B.Fab")
 			(hide yes)
@@
 		)
 		(property "Description" "Resistor"
-			(at 0 0 360)
+			(at 0 0 0)
 			(layer "B.Fab")
 			(hide yes)
@@
 		(tags "resistor handsolder")
 		(property "Reference" "R32"
-			(at 1.45 0 360)
+			(at 1.45 0 0)
 			(layer "B.SilkS")
 			(hide yes)
@@
 		)
 		(property "Value" "10k"
-			(at 0 -1.43 360)
+			(at 0 -1.43 0)
 			(layer "B.Fab")
 			(hide yes)
@@
 		)
 		(property "Footprint" "kicad-mza:0603"
-			(at 0.175 -1.5 360)
+			(at 0.175 -1.5 0)
 			(layer "B.Fab")
 			(hide yes)
@@
 		)
 		(property "Datasheet" ""
-			(at 0 0 360)
+			(at 0 0 0)
 			(layer "B.Fab")
 			(hide yes)
@@
 		)
 		(property "Description" "Resistor"
-			(at 0 0 360)
+			(at 0 0 0)
 			(layer "B.Fab")
 			(hide yes)
@@
 		(tags "resistor handsolder")
 		(property "Reference" "R64"
-			(at 1.45 0 360)
+			(at 1.45 0 0)
 			(layer "B.SilkS")
 			(hide yes)
@@
 		)
 		(property "Value" "10k"
-			(at 0 -1.43 360)
+			(at 0 -1.43 0)
 			(layer "B.Fab")
 			(hide yes)
@@
 		)
 		(property "Footprint" "kicad-mza:0603"
-			(at 0.175 -1.5 360)
+			(at 0.175 -1.5 0)
 			(layer "B.Fab")
 			(hide yes)
@@
 		)
 		(property "Datasheet" ""
-			(at 0 0 360)
+			(at 0 0 0)
 			(layer "B.Fab")
 			(hide yes)
@@
 		)
 		(property "Description" "Resistor"
-			(at 0 0 360)
+			(at 0 0 0)
 			(layer "B.Fab")
 			(hide yes)
@@
 		(tags "resistor handsolder")
 		(property "Reference" "R31"
-			(at 1.45 0 360)
+			(at 1.45 0 0)
 			(layer "B.SilkS")
 			(hide yes)
@@
 		)
 		(property "Value" "10k"
-			(at 0 -1.43 360)
+			(at 0 -1.43 0)
 			(layer "B.Fab")
 			(hide yes)
@@
 		)
 		(property "Footprint" "kicad-mza:0603"
-			(at 0.175 -1.5 360)
+			(at 0.175 -1.5 0)
 			(layer "B.Fab")
 			(hide yes)
@@
 		)
 		(property "Datasheet" ""
-			(at 0 0 360)
+			(at 0 0 0)
 			(layer "B.Fab")
 			(hide yes)
@@
 		)
 		(property "Description" "Resistor"
-			(at 0 0 360)
+			(at 0 0 0)
 			(layer "B.Fab")
 			(hide yes)
@@
 		)
 	)
-	(gr_text "Jacob Romeo\nVarner Lab\n2024-10-28"
+	(gr_text "IDL_24_032"
+		(at 165.6 65.38 -0)
+		(layer "B.SilkS")
+		(effects
+			(font
+				(size 1.5 1.5)
+				(thickness 0.3)
+				(bold yes)
+			)
+			(justify left bottom mirror)
+		)
+	)
+	(gr_text "Jacob Romeo\nVarner Lab\n2024-11-25"
 		(at 126.9 67.43 0)
 		(layer "F.SilkS")
@@
 	)
 	(via
-		(at 160.4 121.03)
-		(size 0.8)
-		(drill 0.4)
-		(layers "F.Cu" "B.Cu")
-		(net 130)
-	)
-	(via
 		(at 168.9 117.23)
 		(size 0.8)
@@
 	)
 	(via
-		(at 133.05 121.48)
-		(size 0.8)
-		(drill 0.4)
-		(layers "F.Cu" "B.Cu")
-		(net 131)
-	)
-	(via
 		(at 138.34723 101.788168)
 		(size 0.8)
@@
 	)
 	(via
-		(at 149 86.93)
-		(size 0.8)
-		(drill 0.4)
-		(layers "F.Cu" "B.Cu")
-		(free yes)
-		(net 132)
-	)
-	(via
 		(at 160.3 73.88)
 		(size 0.8)
@@
 		(size 0.8)
 		(drill 0.4)
-		(layers "F.Cu" "B.Cu")
-		(net 133)
-	)
-	(via
-		(at 146.65 91.93)
-		(size 0.8)
-		(drill 0.4)
