File: SiPMT revA/SiPMT.revA.kicad_pcb (KiCad board)
At the start: 4 copper layers, 55.6 x 69 mm, 150 parts, among them Q1 MountingHole_Pad, Q2 MountingHole_Pad, Q3 MountingHole_Pad, Q4 MountingHole_Pad

Commit message: Made pcie40-waveforms script, updated TOP-BS
Parts:
- added G***: LOGO, kicad-mza:uhm-logo, F.Cu at (159.0, 70.3)
- added G***: LOGO, kicad-mza:Belle2-LOGO, F.Cu at (135.0, 69.7)
Other:
- board text added: ". ."
- board text added: "GND"
- board text added: "IDL_25_009"
- board text added: "Jacob Romeo Varner Lab 2025-09-21"
- board text removed: "IDL_24_032"
- board text removed: "Jacob Romeo Varner Lab 2024-11-25"
